Commit message: Completed quadruped

File: body.urdf (robot description, URDF)
Before this commit: robot robot, 3 links, 2 joints
Links:
- added link LeftLeg, mass 1; collision box size=1 0.2 0.2; visual box size=1 0.2 0.2
- added link LowerBackLeg, mass 1; collision box size=0.2 0.2 1; visual box size=0.2 0.2 1
- added link LowerFrontLeg, mass 1; collision box size=0.2 0.2 1; visual box size=0.2 0.2 1
- added link LowerLeftLeg, mass 1; collision box size=0.2 0.2 1; visual box size=0.2 0.2 1
- added link LowerRightLeg, mass 1; collision box size=0.2 0.2 1; visual box size=0.2 0.2 1
- added link RightLeg, mass 1; collision box size=1 0.2 0.2; visual box size=1 0.2 0.2
- link BackLeg: geometry collision box size=0.2 1 0.2; visual box size=0.2 1 0.2
- link FrontLeg: geometry collision box size=0.2 1 0.2; visual box size=0.2 1 0.2
Joints:
- added joint BackLeg_LowerBackLeg: type revolute, parent BackLeg, child LowerBackLeg, origin xyz=0 -0.5 0 rpy=0 0 0, axis 1 0 0, limit lower=-3.14159 upper=3.14159 effort=0.0 velocity=0.0
- added joint FrontLeg_LowerFrontLeg: type revolute, parent FrontLeg, child LowerFrontLeg, origin xyz=0 0.5 0 rpy=0 0 0, axis 1 0 0, limit lower=-3.14159 upper=3.14159 effort=0.0 velocity=0.0
- added joint LeftLeg_LowerleftLeg: type revolute, parent LeftLeg, child LowerLeftLeg, origin xyz=-0.5 0 0 rpy=0 0 0, axis 0 1 0, limit lower=-3.14159 upper=3.14159 effort=0.0 velocity=0.0
- added joint RightLeg_LowerRightLeg: type revolute, parent RightLeg, child LowerRightLeg, origin xyz=0.5 0 0 rpy=0 0 0, axis 0 1 0, limit lower=-3.14159 upper=3.14159 effort=0.0 velocity=0.0
- added joint Torso_LeftLeg: type revolute, parent Torso, child LeftLeg, origin xyz=-0.5 0 1 rpy=0 0 0, axis 0 1 0, limit lower=-3.14159 upper=3.14159 effort=0.0 velocity=0.0
- added joint Torso_RightLeg: type revolute, parent Torso, child RightLeg, origin xyz=0.5 0 1 rpy=0 0 0, axis 0 1 0, limit lower=-3.14159 upper=3.14159 effort=0.0 velocity=0.0
- joint Torso_BackLeg: axis 0 1 0 -> 1 0 0; origin xyz=1 0 1 rpy=0 0 0 -> xyz=0 -0.5 1 rpy=0 0 0
- joint Torso_FrontLeg: axis 0 1 0 -> 1 0 0; origin xyz=2 0 1 rpy=0 0 0 -> xyz=0 0.5 1 rpy=0 0 0

Commit message: Started daddy long legs project

File: body.urdf (robot description, URDF)
Before this commit: robot robot, 9 links, 8 joints
Links:
- link BackLeg: geometry collision box size=0.2 0.5616240448126326 0.2; visual box size=0.2 0.5616240448126326 0.2
- link FrontLeg: geometry collision box size=0.2 0.216271178647919 0.2; visual box size=0.2 0.216271178647919 0.2
- link LeftLeg: geometry collision box size=1.5179311461881584 0.2 0.2; visual box size=1.5179311461881584 0.2 0.2
- link LowerBackLeg: geometry collision box size=0.2 0.2 1.694208815676067; visual box size=0.2 0.2 1.694208815676067
- link LowerFrontLeg: geometry collision box size=0.2 0.2 1.788081035585855; visual box size=0.2 0.2 1.788081035585855
- link LowerLeftLeg: geometry collision box size=0.2 0.2 1.2726237121847566; visual box size=0.2 0.2 1.2726237121847566
- link LowerRightLeg: geometry collision box size=0.2 0.2 0.01975225258840929; visual box size=0.2 0.2 0.01975225258840929
- link RightLeg: geometry collision box size=1.6103556446372527 0.2 0.2; visual box size=1.6103556446372527 0.2 0.2

Commit message: Completed Daddy long legs

File: body.urdf (robot description, URDF)
Before this commit: robot robot, 9 links, 8 joints
Links:
- link BackLeg: geometry collision box size=0.2 1.3863418392379196 0.2; visual box size=0.2 1.3863418392379196 0.2
- link FrontLeg: geometry collision box size=0.2 1.3863418392379196 0.2; visual box size=0.2 1.3863418392379196 0.2
- link LeftLeg: geometry collision box size=1.3863418392379196 0.2 0.2; visual box size=1.3863418392379196 0.2 0.2
- link LowerBackLeg: geometry collision box size=0.2 0.2 1.4370049075394724; visual box size=0.2 0.2 1.4370049075394724
- link LowerFrontLeg: geometry collision box size=0.2 0.2 1.4370049075394724; visual box size=0.2 0.2 1.4370049075394724
- link LowerLeftLeg: geometry collision box size=0.2 0.2 1.4370049075394724; visual box size=0.2 0.2 1.4370049075394724
- link LowerRightLeg: geometry collision box size=0.2 0.2 1.4370049075394724; visual box size=0.2 0.2 1.4370049075394724
- link RightLeg: geometry collision box size=1.3863418392379196 0.2 0.2; visual box size=1.3863418392379196 0.2 0.2
Joints:
- joint BackLeg_LowerBackLeg: origin xyz=0 -0.5 0 rpy=0 0 0 -> xyz=0 -self.lengths[0,0] self.lengths[0,1] rpy=0 0 0
- joint FrontLeg_LowerFrontLeg: origin xyz=0 0.5 0 rpy=0 0 0 -> xyz=0 self.lengths[0,0] self.lengths[0,1] rpy=0 0 0
- joint LeftLeg_LowerleftLeg: origin xyz=-0.5 0 0 rpy=0 0 0 -> xyz=-self.lengths[0,0] 0 self.lengths[0,1] rpy=0 0 0
- joint RightLeg_LowerRightLeg: origin xyz=0.5 0 0 rpy=0 0 0 -> xyz=self.lengths[0,0] 0 self.lengths[0,1] rpy=0 0 0
- joint Torso_BackLeg: origin xyz=0 -0.5 1 rpy=0 0 0 -> xyz=0 -0.5 self.lengths[0,1] rpy=0 0 0
- joint Torso_FrontLeg: origin xyz=0 0.5 1 rpy=0 0 0 -> xyz=0 0.5 self.lengths[0,1] rpy=0 0 0
- joint Torso_LeftLeg: origin xyz=-0.5 0 1 rpy=0 0 0 -> xyz=-0.5 0 self.lengths[0,1] rpy=0 0 0
- joint Torso_RightLeg: origin xyz=0.5 0 1 rpy=0 0 0 -> xyz=0.5 0 self.lengths[0,1] rpy=0 0 0

Commit message: Finished Daddy Long legs

File: body.urdf (robot description, URDF)
Before this commit: robot robot, 9 links, 8 joints
Links:
- link BackLeg: geometry collision box size=0.2 1.2148022610267728 0.2; visual box size=0.2 1.2148022610267728 0.2
- link FrontLeg: geometry collision box size=0.2 1.2148022610267728 0.2; visual box size=0.2 1.2148022610267728 0.2
- link LeftLeg: geometry collision box size=1.2148022610267728 0.2 0.2; visual box size=1.2148022610267728 0.2 0.2
- link LowerBackLeg: geometry collision box size=0.2 0.2 1.9071853462131418; visual box size=0.2 0.2 1.9071853462131418
- link LowerFrontLeg: geometry collision box size=0.2 0.2 1.9071853462131418; visual box size=0.2 0.2 1.9071853462131418
- link LowerLeftLeg: geometry collision box size=0.2 0.2 1.9071853462131418; visual box size=0.2 0.2 1.9071853462131418
- link LowerRightLeg: geometry collision box size=0.2 0.2 1.9071853462131418; visual box size=0.2 0.2 1.9071853462131418
- link RightLeg: geometry collision box size=1.2148022610267728 0.2 0.2; visual box size=1.2148022610267728 0.2 0.2
Joints:
- joint BackLeg_LowerBackLeg: origin xyz=0 -self.lengths[0,0] self.lengths[0,1] rpy=0 0 0 -> xyz=0 -1.2148022610267728 0 rpy=0 0 0
- joint FrontLeg_LowerFrontLeg: origin xyz=0 self.lengths[0,0] self.lengths[0,1] rpy=0 0 0 -> xyz=0 1.2148022610267728 0 rpy=0 0 0
- joint LeftLeg_LowerleftLeg: origin xyz=-self.lengths[0,0] 0 self.lengths[0,1] rpy=0 0 0 -> xyz=-1.2148022610267728 0 0 rpy=0 0 0
- joint RightLeg_LowerRightLeg: origin xyz=self.lengths[0,0] 0 self.lengths[0,1] rpy=0 0 0 -> xyz=1.2148022610267728 0 0 rpy=0 0 0
- joint Torso_BackLeg: origin xyz=0 -0.5 self.lengths[0,1] rpy=0 0 0 -> xyz=0 -0.5 1.9071853462131418 rpy=0 0 0
- joint Torso_FrontLeg: origin xyz=0 0.5 self.lengths[0,1] rpy=0 0 0 -> xyz=0 0.5 1.9071853462131418 rpy=0 0 0
- joint Torso_LeftLeg: origin xyz=-0.5 0 self.lengths[0,1] rpy=0 0 0 -> xyz=-0.5 0 1.9071853462131418 rpy=0 0 0
- joint Torso_RightLeg: origin xyz=0.5 0 self.lengths[0,1] rpy=0 0 0 -> xyz=0.5 0 1.9071853462131418 rpy=0 0 0

Commit message: Changed fitness function

File: body.urdf (robot description, URDF)
Before this commit: robot robot, 9 links, 8 joints
Links:
- link BackLeg: geometry collision box size=0.2 1 0.2; visual box size=0.2 1 0.2
- link FrontLeg: geometry collision box size=0.2 1 0.2; visual box size=0.2 1 0.2
- link LeftLeg: geometry collision box size=1 0.2 0.2; visual box size=1 0.2 0.2
- link LowerBackLeg: geometry collision box size=0.2 0.2 1; visual box size=0.2 0.2 1
- link LowerFrontLeg: geometry collision box size=0.2 0.2 1; visual box size=0.2 0.2 1
- link LowerLeftLeg: geometry collision box size=0.2 0.2 1; visual box size=0.2 0.2 1
- link LowerRightLeg: geometry collision box size=0.2 0.2 1; visual box size=0.2 0.2 1
- link RightLeg: geometry collision box size=1 0.2 0.2; visual box size=1 0.2 0.2

Commit message: Saved fintess matrix to file

File: body.urdf (robot description, URDF)
Before this commit: robot robot, 9 links, 8 joints
Links:
- link BackLeg: geometry collision box size=0.2 1.064071070589912 0.2; visual box size=0.2 1.064071070589912 0.2
- link FrontLeg: geometry collision box size=0.2 1.064071070589912 0.2; visual box size=0.2 1.064071070589912 0.2
- link LeftLeg: geometry collision box size=1.064071070589912 0.2 0.2; visual box size=1.064071070589912 0.2 0.2
- link LowerBackLeg: geometry collision box size=0.2 0.2 1.0465841571366545; visual box size=0.2 0.2 1.0465841571366545
- link LowerFrontLeg: geometry collision box size=0.2 0.2 1.0465841571366545; visual box size=0.2 0.2 1.0465841571366545
- link LowerLeftLeg: geometry collision box size=0.2 0.2 1.0465841571366545; visual box size=0.2 0.2 1.0465841571366545
- link LowerRightLeg: geometry collision box size=0.2 0.2 1.0465841571366545; visual box size=0.2 0.2 1.0465841571366545
- link RightLeg: geometry collision box size=1.064071070589912 0.2 0.2; visual box size=1.064071070589912 0.2 0.2
Joints:
- joint BackLeg_LowerBackLeg: origin xyz=0 -1.2148022610267728 0 rpy=0 0 0 -> xyz=0 -1.064071070589912 0 rpy=0 0 0
- joint FrontLeg_LowerFrontLeg: origin xyz=0 1.2148022610267728 0 rpy=0 0 0 -> xyz=0 1.064071070589912 0 rpy=0 0 0
- joint LeftLeg_LowerleftLeg: origin xyz=-1.2148022610267728 0 0 rpy=0 0 0 -> xyz=-1.064071070589912 0 0 rpy=0 0 0
- joint RightLeg_LowerRightLeg: origin xyz=1.2148022610267728 0 0 rpy=0 0 0 -> xyz=1.064071070589912 0 0 rpy=0 0 0
- joint Torso_BackLeg: origin xyz=0 -0.5 1.9071853462131418 rpy=0 0 0 -> xyz=0 -0.5 1.0465841571366545 rpy=0 0 0
- joint Torso_FrontLeg: origin xyz=0 0.5 1.9071853462131418 rpy=0 0 0 -> xyz=0 0.5 1.0465841571366545 rpy=0 0 0
- joint Torso_LeftLeg: origin xyz=-0.5 0 1.9071853462131418 rpy=0 0 0 -> xyz=-0.5 0 1.0465841571366545 rpy=0 0 0
- joint Torso_RightLeg: origin xyz=0.5 0 1.9071853462131418 rpy=0 0 0 -> xyz=0.5 0 1.0465841571366545 rpy=0 0 0
